Commit message: Add files via upload

File: robotic_arm/urdf/robotic_arm.urdf (robot description, URDF)
Before this commit: robot robotic_arm, 4 links, 3 joints
Links:
- removed link humerus
- removed link turntable
- link base_link: geometry collision mesh filename=package://robotic_arm/meshes/base.STL scale=0.1 0.1 0.1; visual mesh filename=package://robotic_arm/meshes/base.STL scale=0.1 0.1 0.1
Joints:
- removed joint plate_to_turntable
- removed joint turntable_to_humerus_joint

Commit message: fix the assembly origins

File: robotic_arm/urdf/robotic_arm.urdf (robot description, URDF)
Before this commit: robot robotic_arm, 2 links, 1 joints
Links:
- added link revolve_motor, mass 0.1; collision mesh filename=package://robotic_arm/meshes/AX-12A.STL scale=0.001 0.001 0.001; visual mesh filename=package://robotic_arm/meshes/AX-12A.STL scale=0.001 0.001 0.001
- link base_link: geometry collision mesh filename=package://robotic_arm/meshes/base.STL scale=0.001 0.001 0.001; visual mesh filename=package://robotic_arm/meshes/base.STL scale=0.001 0.001 0.001
Joints:
- added joint revolvemotor_to_baseplate: type fixed, parent base_link, child revolve_motor, origin xyz=0 0 0.0225
- joint fixed: origin (none) -> xyz=0 0 0.0025 rpy=0 0 0

File: robotic_arm/urdf/robotic_enclosure.urdf (robot description, URDF)
Before this commit: robot robotic_arm, 4 links, 3 joints
Links:
- removed link base_link
- removed link enclosure
- removed link humerus
- removed link turntable
- added link world
Joints:
- removed joint enclosure_to_plate
- removed joint plate_to_turntable
- removed joint turntable_to_humerus_joint
- added joint fixed: type fixed, parent world, child enclosure
